File: companion_computer.kicad_pcb (KiCad board)
At the start: 2 copper layers, 1 part, among them U1 RK3566

Commit message: initial commit
Connections:
- U1 pad 1A10: unconnected-(U1E-DDR_DQ5_B/DDR4_DQU6_B/LPDDR4_DQ5_B/DDR3_DQ21/LPDDR3_DQ3-Pad1A10) -> /LPDDR4_DQ5_B
- U1 pad 1A11: unconnected-(U1E-DDR_DM1_B/DDR4_DML_B/LPDDR4_DM1_B/DDR3_DM3/LPDDR3_DM2-Pad1A11) -> /LPDDR4_DM1_B
- U1 pad 1A7: unconnected-(U1E-DDR_DQ3_B/DDR4_DQU1_B/LPDDR4_DQ3_B/DDR3_DQ19/LPDDR3_DQ4-Pad1A7) -> /LPDDR4_DQ3_B
- U1 pad 1A8: unconnected-(U1E-DDR_DQ2_B/DDR4_DQU3_B/LPDDR4_DQ2_B/DDR3_DQ18/LPDDR3_DQ6-Pad1A8) -> /LPDDR4_DQ2_B
- U1 pad 1A9: unconnected-(U1E-DDR_DQ7_B/DDR4_DQU2_B/LPDDR4_DQ7_B/DDR3_DQ23/LPDDR3_DQ0-Pad1A9) -> /LPDDR4_DQ7_B
- U1 pad 1B10: unconnected-(U1H-VSS_30-Pad1B10) -> GNDREF
- U1 pad 1B11: unconnected-(U1H-VSS_31-Pad1B11) -> GNDREF
- U1 pad 1B15: unconnected-(U1H-VSS_32-Pad1B15) -> GNDREF
- U1 pad 1B19: unconnected-(U1H-VSS_33-Pad1B19) -> GNDREF
- U1 pad 1B8: unconnected-(U1E-DDR_DM0_B/DDR4_DMU_B/LPDDR4_DM0_B/DDR3_DM2/LPDDR3_DM0-Pad1B8) -> /LPDDR4_DM0_B
- U1 pad 1B9: unconnected-(U1E-DDR_DQ6_B/DDR4_DQU4_B/LPDDR4_DQ6_B/DDR3_DQ22/LPDDR3_DQ7-Pad1B9) -> /LPDDR4_DQ6_B
- U1 pad 1C10: unconnected-(U1E-DDR_DQ14_B/DDR4_DQL1_B/LPDDR4_DQ14_B/DDR3_DQ30/LPDDR3_DQ20-Pad1C10) -> /LPDDR4_DQ14_B
- U1 pad 1C12: unconnected-(U1F-VDD_CPU_1-Pad1C12) -> VDD_CPU
- U1 pad 1C14: unconnected-(U1H-VSS_39-Pad1C14) -> GNDREF
- U1 pad 1C16: unconnected-(U1H-VSS_40-Pad1C16) -> GNDREF
- U1 pad 1C18: unconnected-(U1H-VSS_41-Pad1C18) -> GNDREF
- U1 pad 1C4: unconnected-(U1H-VSS_34-Pad1C4) -> GNDREF
- U1 pad 1C5: unconnected-(U1H-VSS_35-Pad1C5) -> GNDREF
- U1 pad 1C6: unconnected-(U1H-VSS_36-Pad1C6) -> GNDREF
- U1 pad 1C8: unconnected-(U1H-VSS_37-Pad1C8) -> GNDREF
- U1 pad 1C9: unconnected-(U1H-VSS_38-Pad1C9) -> GNDREF
- U1 pad 1D1: unconnected-(U1H-VSS_42-Pad1D1) -> GNDREF
- U1 pad 1D10: unconnected-(U1H-VSS_44-Pad1D10) -> GNDREF
- U1 pad 1D11: unconnected-(U1F-VDD_CPU_2-Pad1D11) -> VDD_CPU
- U1 pad 1D12: unconnected-(U1F-VDD_CPU_3-Pad1D12) -> VDD_CPU
- U1 pad 1D14: unconnected-(U1H-VSS_45-Pad1D14) -> GNDREF
- U1 pad 1D3: unconnected-(U1H-VSS_43-Pad1D3) -> GNDREF
- U1 pad 1D4: unconnected-(U1E-DDR_AVSS-Pad1D4) -> GNDREF
- U1 pad 1D5: unconnected-(U1E-DDRPHY_VDDQ_1-Pad1D5) -> VCC_DDR
- U1 pad 1D6: unconnected-(U1E-DDRPHY_VDDQ_2-Pad1D6) -> VCC_DDR
- U1 pad 1D7: unconnected-(U1E-DDRPHY_VDDQ_3-Pad1D7) -> VCC_DDR
- U1 pad 1D8: unconnected-(U1E-DDRPHY_VDDQ_4-Pad1D8) -> VCC_DDR
- U1 pad 1D9: unconnected-(U1E-DDRPHY_VDDQ_5-Pad1D9) -> VCC_DDR
- U1 pad 1E1: unconnected-(U1E-DDR_DQ7_A/DDR4_DQL1_A/LPDDR4_DQ7_A/DDR3_DQ7/LPDDR3_DQ11-Pad1E1) -> /LPDDR4_DQ7_A
- U1 pad 1E10: unconnected-(U1H-VSS_48-Pad1E10) -> GNDREF
- U1 pad 1E11: unconnected-(U1F-VDD_CPU_4-Pad1E11) -> VDD_CPU
- U1 pad 1E12: unconnected-(U1F-VDD_CPU_5-Pad1E12) -> VDD_CPU
- U1 pad 1E13: unconnected-(U1F-VDD_CPU_6-Pad1E13) -> VDD_CPU
- U1 pad 1E14: unconnected-(U1H-VSS_49-Pad1E14) -> GNDREF
- U1 pad 1E15: unconnected-(U1H-VSS_50-Pad1E15) -> GNDREF
- U1 pad 1E17: unconnected-(U1H-VSS_51-Pad1E17) -> GNDREF
- U1 pad 1E2: unconnected-(U1E-DDR_DM0_A/DDR4_DML_A/LPDDR4_DM0_A/DDR3_DM0/LPDDR3_DM1-Pad1E2) -> /LPDDR4_DM0_A
- U1 pad 1E3: unconnected-(U1H-VSS_46-Pad1E3) -> GNDREF
- U1 pad 1E4: unconnected-(U1E-DDRPHY_VDDQ_6-Pad1E4) -> VCC_DDR
- U1 pad 1E6: unconnected-(U1E-DDRPHY_VDDQL_1-Pad1E6) -> VCC0V6_DDR
- U1 pad 1E7: unconnected-(U1E-DDRPHY_VDDQL_2-Pad1E7) -> VCC0V6_DDR
- U1 pad 1E8: unconnected-(U1H-VSS_47-Pad1E8) -> GNDREF
- U1 pad 1E9: unconnected-(U1E-DDRPHY_VDDQL_3-Pad1E9) -> VCC0V6_DDR
- U1 pad 1F1: unconnected-(U1E-DDR_DQ14_A/DDR4_DQU6_A/LPDDR4_DQ14_A/DDR3_DQ14/LPDDR3_DQ30-Pad1F1) -> /LPDDR4_DQ14_A
- U1 pad 1F10: unconnected-(U1H-VSS_56-Pad1F10) -> GNDREF
- U1 pad 1F11: unconnected-(U1F-VDD_CPU_7-Pad1F11) -> VDD_CPU
- U1 pad 1F12: unconnected-(U1F-VDD_CPU_8-Pad1F12) -> VDD_CPU
- U1 pad 1F13: unconnected-(U1F-VDD_CPU_9-Pad1F13) -> VDD_CPU
- U1 pad 1F14: unconnected-(U1F-VDD_CPU_10-Pad1F14) -> VDD_CPU
- U1 pad 1F15: unconnected-(U1H-VSS_57-Pad1F15) -> GNDREF
- U1 pad 1F16: unconnected-(U1H-VSS_58-Pad1F16) -> GNDREF
- U1 pad 1F2: unconnected-(U1E-DDR_DQ13_A/DDR4_DQU4_A/LPDDR4_DQ13_A/DDR3_DQ13/LPDDR3_DQ31-Pad1F2) -> /LPDDR4_DQ13_A
- U1 pad 1F20: unconnected-(U1G-AVSS1_6-Pad1F20) -> GNDREF
- U1 pad 1F3: unconnected-(U1E-DDR_RZQ-Pad1F3) -> Net-(U1E-DDR_RZQ)
- U1 pad 1F4: unconnected-(U1E-DDRPHY_VDDQ_7-Pad1F4) -> VCC_DDR
- U1 pad 1F5: unconnected-(U1E-DDRPHY_VDDQL_4-Pad1F5) -> VCC0V6_DDR
- U1 pad 1F6: unconnected-(U1H-VSS_52-Pad1F6) -> GNDREF
- U1 pad 1F7: unconnected-(U1H-VSS_53-Pad1F7) -> GNDREF
- U1 pad 1F8: unconnected-(U1H-VSS_54-Pad1F8) -> GNDREF
- U1 pad 1F9: unconnected-(U1H-VSS_55-Pad1F9) -> GNDREF
- U1 pad 1G1: unconnected-(U1E-DDR_DM1_A/DDR4_DMU_A/LPDDR4_DM1_A/DDR3_DM1/LPDDR3_DM3-Pad1G1) -> /LPDDR4_DM1_A
- U1 pad 1G10: unconnected-(U1H-VSS_64-Pad1G10) -> GNDREF
- U1 pad 1G11: unconnected-(U1H-VSS_65-Pad1G11) -> GNDREF
- U1 pad 1G12: unconnected-(U1H-VSS_66-Pad1G12) -> GNDREF
- U1 pad 1G13: unconnected-(U1F-VDD_CPU_11-Pad1G13) -> VDD_CPU
- U1 pad 1G14: unconnected-(U1I-VSS_67-Pad1G14) -> GNDREF
- U1 pad 1G15: unconnected-(U1F-VDD_NPU_1-Pad1G15) -> VDD_GPU_NPU
- U1 pad 1G16: unconnected-(U1G-AVSS1_7-Pad1G16) -> GNDREF
- U1 pad 1G18: unconnected-(U1G-AVSS1_8-Pad1G18) -> GNDREF
- U1 pad 1G19: unconnected-(U1G-AVSS1_9-Pad1G19) -> GNDREF
- U1 pad 1G2: unconnected-(U1E-DDR_DQ15_A/DDR4_DQU0_A/LPDDR4_DQ15_A/DDR3_DQ15/LPDDR3_DQ27-Pad1G2) -> /LPDDR4_DQ15_A
- U1 pad 1G20: unconnected-(U1G-AVSS1_10-Pad1G20) -> GNDREF
- U1 pad 1G3: unconnected-(U1H-VSS_59-Pad1G3) -> GNDREF
- U1 pad 1G4: unconnected-(U1E-DDRPHY_VDDQ_8-Pad1G4) -> VCC_DDR
- U1 pad 1G5: unconnected-(U1E-DDRPHY_VDDQL_5-Pad1G5) -> VCC0V6_DDR
- U1 pad 1G6: unconnected-(U1H-VSS_60-Pad1G6) -> GNDREF
- U1 pad 1G7: unconnected-(U1H-VSS_61-Pad1G7) -> GNDREF
- U1 pad 1G8: unconnected-(U1H-VSS_62-Pad1G8) -> GNDREF
- U1 pad 1G9: unconnected-(U1H-VSS_63-Pad1G9) -> GNDREF
- U1 pad 1H1: unconnected-(U1I-VSS_68-Pad1H1) -> GNDREF
- U1 pad 1H10: unconnected-(U1F-VDD_LOGIC_4-Pad1H10) -> VDD_LOGIC
- U1 pad 1H11: unconnected-(U1I-VSS_71-Pad1H11) -> GNDREF
- U1 pad 1H12: unconnected-(U1I-VSS_72-Pad1H12) -> GNDREF
- U1 pad 1H13: unconnected-(U1I-VSS_73-Pad1H13) -> GNDREF
- U1 pad 1H14: unconnected-(U1F-VDD_NPU_2-Pad1H14) -> VDD_GPU_NPU
- U1 pad 1H15: unconnected-(U1F-VDD_NPU_3-Pad1H15) -> VDD_GPU_NPU
- U1 pad 1H2: unconnected-(U1I-VSS_69-Pad1H2) -> GNDREF
- U1 pad 1H6: unconnected-(U1I-VSS_70-Pad1H6) -> GNDREF
- U1 pad 1H7: unconnected-(U1F-VDD_LOGIC_1-Pad1H7) -> VDD_LOGIC
- U1 pad 1H8: unconnected-(U1F-VDD_LOGIC_2-Pad1H8) -> VDD_LOGIC
- U1 pad 1H9: unconnected-(U1F-VDD_LOGIC_3-Pad1H9) -> VDD_LOGIC
- U1 pad 1J1: unconnected-(U1I-VSS_74-Pad1J1) -> GNDREF
- U1 pad 1J10: unconnected-(U1F-VDD_LOGIC_6-Pad1J10) -> VDD_LOGIC
- U1 pad 1J11: unconnected-(U1I-VSS_78-Pad1J11) -> GNDREF
- U1 pad 1J12: unconnected-(U1I-VSS_79-Pad1J12) -> GNDREF
- U1 pad 1J13: unconnected-(U1I-VSS_80-Pad1J13) -> GNDREF
- U1 pad 1J14: unconnected-(U1F-VDD_NPU_4-Pad1J14) -> VDD_GPU_NPU
- U1 pad 1J15: unconnected-(U1F-VDD_NPU_5-Pad1J15) -> VDD_GPU_NPU
- U1 pad 1J16: unconnected-(U1G-AVSS1_11-Pad1J16) -> GNDREF
- U1 pad 1J18: unconnected-(U1G-AVSS1_12-Pad1J18) -> GNDREF
- U1 pad 1J6: unconnected-(U1I-VSS_75-Pad1J6) -> GNDREF
- U1 pad 1J7: unconnected-(U1F-VDD_LOGIC_5-Pad1J7) -> VDD_LOGIC
- U1 pad 1J8: unconnected-(U1I-VSS_76-Pad1J8) -> GNDREF
- U1 pad 1J9: unconnected-(U1I-VSS_77-Pad1J9) -> GNDREF
- U1 pad 1K10: unconnected-(U1F-VDD_LOGIC_8-Pad1K10) -> VDD_LOGIC
- U1 pad 1K11: unconnected-(U1I-VSS_88-Pad1K11) -> GNDREF
- U1 pad 1K12: unconnected-(U1I-VSS_89-Pad1K12) -> GNDREF
- U1 pad 1K13: unconnected-(U1I-VSS_90-Pad1K13) -> GNDREF
- U1 pad 1K14: unconnected-(U1I-VSS_91-Pad1K14) -> GNDREF
- U1 pad 1K15: unconnected-(U1I-VSS_92-Pad1K15) -> GNDREF
- U1 pad 1K18: unconnected-(U1G-AVSS1_13-Pad1K18) -> GNDREF
- U1 pad 1K2: unconnected-(U1I-VSS_81-Pad1K2) -> GNDREF
- U1 pad 1K3: unconnected-(U1I-VSS_82-Pad1K3) -> GNDREF
- U1 pad 1K4: unconnected-(U1I-VSS_83-Pad1K4) -> GNDREF
- U1 pad 1K5: unconnected-(U1I-VSS_84-Pad1K5) -> GNDREF
- U1 pad 1K6: unconnected-(U1I-VSS_85-Pad1K6) -> GNDREF
- U1 pad 1K7: unconnected-(U1F-VDD_LOGIC_7-Pad1K7) -> VDD_LOGIC
- U1 pad 1K8: unconnected-(U1I-VSS_86-Pad1K8) -> GNDREF
- U1 pad 1K9: unconnected-(U1I-VSS_87-Pad1K9) -> GNDREF
- U1 pad 1L10: unconnected-(U1I-VSS_95-Pad1L10) -> GNDREF
- U1 pad 1L11: unconnected-(U1I-VSS_96-Pad1L11) -> GNDREF
- U1 pad 1L12: unconnected-(U1I-VSS_97-Pad1L12) -> GNDREF
- U1 pad 1L13: unconnected-(U1I-VSS_98-Pad1L13) -> GNDREF
- U1 pad 1L14: unconnected-(U1I-VSS_99-Pad1L14) -> GNDREF
- U1 pad 1L15: unconnected-(U1I-VSS_100-Pad1L15) -> GNDREF
- U1 pad 1L19: unconnected-(U1G-AVSS1_14-Pad1L19) -> GNDREF
- U1 pad 1L3: unconnected-(U1I-VSS_93-Pad1L3) -> GNDREF
- U1 pad 1L6: unconnected-(U1I-VSS_94-Pad1L6) -> GNDREF
- U1 pad 1L7: unconnected-(U1F-VDD_LOGIC_9-Pad1L7) -> VDD_LOGIC
- U1 pad 1L8: unconnected-(U1F-VDD_GPU_1-Pad1L8) -> VDD_GPU_NPU
- U1 pad 1L9: unconnected-(U1F-VDD_GPU_2-Pad1L9) -> VDD_GPU_NPU
- U1 pad 1M10: unconnected-(U1I-VSS_105-Pad1M10) -> GNDREF
- U1 pad 1M11: unconnected-(U1I-VSS_106-Pad1M11) -> GNDREF
- U1 pad 1M12: unconnected-(U1I-VSS_107-Pad1M12) -> GNDREF
- U1 pad 1M13: unconnected-(U1I-VSS_108-Pad1M13) -> GNDREF
- U1 pad 1M14: unconnected-(U1I-VSS_109-Pad1M14) -> GNDREF
- U1 pad 1M15: unconnected-(U1I-VSS_110-Pad1M15) -> GNDREF
- U1 pad 1M16: unconnected-(U1I-VSS_111-Pad1M16) -> GNDREF
- U1 pad 1M17: unconnected-(U1I-VSS_112-Pad1M17) -> GNDREF
- U1 pad 1M18: unconnected-(U1G-TVSS-Pad1M18) -> GNDREF
- U1 pad 1M20: unconnected-(U1I-VSS_113-Pad1M20) -> GNDREF
- U1 pad 1M3: unconnected-(U1I-VSS_101-Pad1M3) -> GNDREF
- U1 pad 1M4: unconnected-(U1I-VSS_102-Pad1M4) -> GNDREF
- U1 pad 1M5: unconnected-(U1I-VSS_103-Pad1M5) -> GNDREF
- U1 pad 1M6: unconnected-(U1I-VSS_104-Pad1M6) -> GNDREF
- U1 pad 1M7: unconnected-(U1F-VDD_GPU_3-Pad1M7) -> VDD_GPU_NPU
- U1 pad 1M8: unconnected-(U1F-VDD_GPU_4-Pad1M8) -> VDD_GPU_NPU
- U1 pad 1M9: unconnected-(U1F-VDD_GPU_5-Pad1M9) -> VDD_GPU_NPU
- U1 pad 1N11: unconnected-(U1G-AVSS_9-Pad1N11) -> GNDREF
- U1 pad 1N12: unconnected-(U1G-AVSS_10-Pad1N12) -> GNDREF
- U1 pad 1N3: unconnected-(U1I-VSS_114-Pad1N3) -> GNDREF
- U1 pad 1N4: unconnected-(U1I-VSS_115-Pad1N4) -> GNDREF
- U1 pad 1N7: unconnected-(U1I-VSS_116-Pad1N7) -> GNDREF
- U1 pad 1P1: unconnected-(U1I-VSS_117-Pad1P1) -> GNDREF
- U1 pad 1P10: unconnected-(U1G-AVSS_12-Pad1P10) -> GNDREF
- U1 pad 1P14: unconnected-(U1G-AVSS_13-Pad1P14) -> GNDREF
- U1 pad 1P15: unconnected-(U1I-VSS_121-Pad1P15) -> GNDREF
- U1 pad 1P5: unconnected-(U1I-VSS_118-Pad1P5) -> GNDREF
- U1 pad 1P6: unconnected-(U1I-VSS_119-Pad1P6) -> GNDREF
- U1 pad 1P7: unconnected-(U1I-VSS_120-Pad1P7) -> GNDREF
- U1 pad 1P8: unconnected-(U1G-AVSS_11-Pad1P8) -> GNDREF
- U1 pad 1R11: unconnected-(U1G-AVSS_16-Pad1R11) -> GNDREF
- U1 pad 1R12: unconnected-(U1G-AVSS_17-Pad1R12) -> GNDREF
- U1 pad 1R13: unconnected-(U1G-AVSS_18-Pad1R13) -> GNDREF
- U1 pad 1R14: unconnected-(U1G-AVSS_19-Pad1R14) -> GNDREF
- U1 pad 1R15: unconnected-(U1G-AVSS_20-Pad1R15) -> GNDREF
- U1 pad 1R3: unconnected-(U1I-VSS_122-Pad1R3) -> GNDREF
- U1 pad 1R4: unconnected-(U1I-VSS_123-Pad1R4) -> GNDREF
- U1 pad 1R5: unconnected-(U1I-VSS_124-Pad1R5) -> GNDREF
- U1 pad 1R6: unconnected-(U1I-VSS_125-Pad1R6) -> GNDREF
- U1 pad 1R7: unconnected-(U1I-VSS_126-Pad1R7) -> GNDREF
- U1 pad 1R8: unconnected-(U1G-AVSS_14-Pad1R8) -> GNDREF
- U1 pad 1R9: unconnected-(U1G-AVSS_15-Pad1R9) -> GNDREF
- U1 pad 1T10: unconnected-(U1G-AVSS_24-Pad1T10) -> GNDREF
- U1 pad 1T11: unconnected-(U1G-AVSS_25-Pad1T11) -> GNDREF
- U1 pad 1T12: unconnected-(U1G-AVSS_26-Pad1T12) -> GNDREF
- U1 pad 1T13: unconnected-(U1G-AVSS_27-Pad1T13) -> GNDREF
- U1 pad 1T14: unconnected-(U1G-AVSS_28-Pad1T14) -> GNDREF
- U1 pad 1T15: unconnected-(U1G-AVSS_29-Pad1T15) -> GNDREF
- U1 pad 1T16: unconnected-(U1G-AVSS_30-Pad1T16) -> GNDREF
- U1 pad 1T17: unconnected-(U1G-AVSS_31-Pad1T17) -> GNDREF
- U1 pad 1T3: unconnected-(U1I-VSS_127-Pad1T3) -> GNDREF
- U1 pad 1T5: unconnected-(U1I-VSS_128-Pad1T5) -> GNDREF
- U1 pad 1T7: unconnected-(U1G-AVSS_21-Pad1T7) -> GNDREF
- U1 pad 1T8: unconnected-(U1G-AVSS_22-Pad1T8) -> GNDREF
- U1 pad 1T9: unconnected-(U1G-AVSS_23-Pad1T9) -> GNDREF
- U1 pad 1U12: unconnected-(U1G-AVSS_32-Pad1U12) -> GNDREF
- U1 pad 1U13: unconnected-(U1G-AVSS_33-Pad1U13) -> GNDREF
- U1 pad 1U15: unconnected-(U1G-AVSS_34-Pad1U15) -> GNDREF
- U1 pad 1U17: unconnected-(U1G-AVSS_35-Pad1U17) -> GNDREF
- U1 pad 1U2: unconnected-(U1I-VSS_129-Pad1U2) -> GNDREF
- U1 pad 1V1: unconnected-(U1I-VSS_130-Pad1V1) -> GNDREF
- U1 pad 1V12: unconnected-(U1G-AVSS_37-Pad1V12) -> GNDREF
- U1 pad 1V13: unconnected-(U1G-AVSS_38-Pad1V13) -> GNDREF
- U1 pad 1V18: unconnected-(U1G-AVSS_39-Pad1V18) -> GNDREF
- U1 pad 1V4: unconnected-(U1I-VSS_131-Pad1V4) -> GNDREF
- U1 pad 1V7: unconnected-(U1G-AVSS_36-Pad1V7) -> GNDREF
- U1 pad A1: unconnected-(U1H-VSS_1-PadA1) -> GNDREF
- U1 pad A12: unconnected-(U1E-DDR_DQS0N_B/DDR4_DQSU_N_B/LPDDR4_DQS0N_B/DDR3_DQS2N/LPDDR3_DQS0N-PadA12) -> /LPDDR4_DQS0N_B
- U1 pad A13: unconnected-(U1E-DDR_DQS0P_B/DDR4_DQSU_P_B/LPDDR4_DQS0P_B/DDR3_DQS2P/LPDDR3_DQS0P-PadA13) -> /LPDDR4_DQS0P_B
- U1 pad A15: unconnected-(U1E-DDR_DQ12_B/DDR4_DQL7_B/LPDDR4_DQ12_B/DDR3_DQ28/LPDDR3_DQ16-PadA15) -> /LPDDR4_DQ12_B
- U1 pad A17: unconnected-(U1E-DDR_DQS1P_B/DDR4_DQSL_P_B/LPDDR4_DQS1P_B/DDR3_DQS3P/LPDDR3_DQS2P-PadA17) -> /LPDDR4_DQS1P_B
- U1 pad A19: unconnected-(U1E-DDR_DQ9_B/DDR4_DQL2_B/LPDDR4_DQ9_B/DDR3_DQ25/LPDDR3_DQ19-PadA19) -> /LPDDR4_DQ9_B
- U1 pad A2: unconnected-(U1H-VSS_2-PadA2) -> GNDREF
- U1 pad A20: unconnected-(U1E-DDR_DQ10_B/DDR4_DQL4_B/LPDDR4_DQ10_B/DDR3_DQ26/LPDDR3_DQ22-PadA20) -> /LPDDR4_DQ10_B
- U1 pad A38: unconnected-(U1H-VSS_3-PadA38) -> GNDREF
- U1 pad AA2: unconnected-(U1H-VSS_18-PadAA2) -> GNDREF
- U1 pad AC37: unconnected-(U1H-VSS_24-PadAC37) -> GNDREF
- U1 pad AD2: unconnected-(U1H-VSS_19-PadAD2) -> GNDREF
- U1 pad AE37: unconnected-(U1H-VSS_25-PadAE37) -> GNDREF
- U1 pad AH37: unconnected-(U1H-VSS_26-PadAH37) -> GNDREF
- U1 pad AL37: unconnected-(U1H-VSS_27-PadAL37) -> GNDREF
- U1 pad AP13: unconnected-(U1G-AVSS_1-PadAP13) -> GNDREF
- U1 pad AP16: unconnected-(U1G-AVSS_2-PadAP16) -> GNDREF
- U1 pad AP19: unconnected-(U1G-AVSS_3-PadAP19) -> GNDREF
- U1 pad AP2: unconnected-(U1H-VSS_20-PadAP2) -> GNDREF
- U1 pad AP22: unconnected-(U1G-AVSS_4-PadAP22) -> GNDREF
- U1 pad AP25: unconnected-(U1G-AVSS_5-PadAP25) -> GNDREF
- U1 pad AP28: unconnected-(U1G-AVSS_6-PadAP28) -> GNDREF
- U1 pad AP31: unconnected-(U1G-AVSS_7-PadAP31) -> GNDREF
- U1 pad AP34: unconnected-(U1G-AVSS_8-PadAP34) -> GNDREF
- U1 pad AP37: unconnected-(U1H-VSS_28-PadAP37) -> GNDREF
- U1 pad AP8: unconnected-(U1H-VSS_22-PadAP8) -> GNDREF
- U1 pad AR1: unconnected-(U1H-VSS_21-PadAR1) -> GNDREF
- U1 pad AR38: unconnected-(U1H-VSS_29-PadAR38) -> GNDREF
- U1 pad B1: unconnected-(U1H-VSS_4-PadB1) -> GNDREF
- U1 pad B10: unconnected-(U1E-DDR_DQ1_B/DDR4_DQU5_B/LPDDR4_DQ1_B/DDR3_DQ17/LPDDR3_DQ5-PadB10) -> /LPDDR4_DQ1_B
- U1 pad B11: unconnected-(U1H-VSS_7-PadB11) -> GNDREF
- U1 pad B12: unconnected-(U1E-DDR_DQ0_B/DDR4_DQU7_B/LPDDR4_DQ0_B/DDR3_DQ16/LPDDR3_DQ1-PadB12) -> /LPDDR4_DQ0_B
- U1 pad B13: unconnected-(U1E-DDR_DQ4_B/DDR4_DQU0_B/LPDDR4_DQ4_B/DDR3_DQ20/LPDDR3_DQ2-PadB13) -> /LPDDR4_DQ4_B
- U1 pad B14: unconnected-(U1H-VSS_8-PadB14) -> GNDREF
- U1 pad B15: unconnected-(U1E-DDR_DQ13_B/DDR4_DQL5_B/LPDDR4_DQ13_B/DDR3_DQ29/LPDDR3_DQ17-PadB15) -> /LPDDR4_DQ13_B
- U1 pad B16: unconnected-(U1E-DDR_DQ15_B/DDR4_DQL3_B/LPDDR4_DQ15_B/DDR3_DQ31/LPDDR3_DQ21-PadB16) -> /LPDDR4_DQ15_B
- U1 pad B17: unconnected-(U1E-DDR_DQS1N_B/DDR4_DQSL_N_B/LPDDR4_DQS1N_B/DDR3_DQS3N/LPDDR3_DQS2N-PadB17) -> /LPDDR4_DQS1N_B
- U1 pad B18: unconnected-(U1H-VSS_9-PadB18) -> GNDREF
- U1 pad B19: unconnected-(U1E-DDR_DQ8_B/DDR4_DQL0_B/LPDDR4_DQ8_B/DDR3_DQ24/LPDDR3_DQ18-PadB19) -> /LPDDR4_DQ8_B
- U1 pad B2: unconnected-(U1H-VSS_5-PadB2) -> GNDREF
- U1 pad B20: unconnected-(U1E-DDR_DQ11_B/DDR4_DQL6_B/LPDDR4_DQ11_B/DDR3_DQ27/LPDDR3_DQ23-PadB20) -> /LPDDR4_DQ11_B
- U1 pad B21: unconnected-(U1H-VSS_10-PadB21) -> GNDREF
- U1 pad B28: unconnected-(U1H-VSS_11-PadB28) -> GNDREF
- U1 pad B31: unconnected-(U1H-VSS_12-PadB31) -> GNDREF
- U1 pad B6: unconnected-(U1H-VSS_6-PadB6) -> GNDREF
- U1 pad D2: unconnected-(U1H-VSS_13-PadD2) -> GNDREF
- U1 pad E1: unconnected-(U1E-DDR_DQ3_A/DDR4_DQL6_A/LPDDR4_DQ3_A/DDR3_DQ3/LPDDR3_DQ9-PadE1) -> /LPDDR4_DQ3_A
- U1 pad E37: unconnected-(U1H-VSS_23-PadE37) -> GNDREF
- U1 pad F1: unconnected-(U1E-DDR_DQ2_A/DDR4_DQL4_A/LPDDR4_DQ2_A/DDR3_DQ2/LPDDR3_DQ10-PadF1) -> /LPDDR4_DQ2_A
- U1 pad F2: unconnected-(U1E-DDR_DQ1_A/DDR4_DQL2_A/LPDDR4_DQ1_A/DDR3_DQ1/LPDDR3_DQ14-PadF2) -> /LPDDR4_DQ1_A
- U1 pad G2: unconnected-(U1E-DDR_DQ0_A/DDR4_DQL0_A/LPDDR4_DQ0_A/DDR3_DQ0/LPDDR3_DQ15-PadG2) -> /LPDDR4_DQ0_A
- U1 pad H1: unconnected-(U1E-DDR_DQS0N_A/DDR4_DQSL_N_A/LPDDR4_DQS0N_A/DDR3_DQS0N/LPDDR3_DQS1N-PadH1) -> /LPDDR4_DQS0N_A
- U1 pad H2: unconnected-(U1E-DDR_DQS0P_A/DDR4_DQSL_P_A/LPDDR4_DQS0P_A/DDR3_DQS0P/LPDDR3_DQS1P-PadH2) -> /LPDDR4_DQS0P_A
- U1 pad H37: unconnected-(U1G-AVSS1_1-PadH37) -> GNDREF
- U1 pad J2: unconnected-(U1H-VSS_14-PadJ2) -> GNDREF
- U1 pad K1: unconnected-(U1E-DDR_DQ5_A/DDR4_DQL5_A/LPDDR4_DQ5_A/DDR3_DQ5/LPDDR3_DQ12-PadK1) -> /LPDDR4_DQ5_A
- U1 pad K2: unconnected-(U1E-DDR_DQ6_A/DDR4_DQL3_A/LPDDR4_DQ6_A/DDR3_DQ6/LPDDR3_DQ8-PadK2) -> /LPDDR4_DQ6_A
- U1 pad L2: unconnected-(U1H-VSS_15-PadL2) -> GNDREF
- U1 pad L37: unconnected-(U1G-AVSS1_2-PadL37) -> GNDREF
- U1 pad M1: unconnected-(U1E-DDR_DQ12_A/DDR4_DQU2_A/LPDDR4_DQ12_A/DDR3_DQ12/LPDDR3_DQ26-PadM1) -> /LPDDR4_DQ12_A
- U1 pad M2: unconnected-(U1E-DDR_DQ4_A/DDR4_DQL7_A/LPDDR4_DQ4_A/DDR3_DQ4/LPDDR3_DQ13-PadM2) -> /LPDDR4_DQ4_A
- U1 pad N1: unconnected-(U1E-DDR_DQS1P_A/DDR4_DQSU_P_A/LPDDR4_DQS1P_A/DDR3_DQS1P/LPDDR3_DQS3P-PadN1) -> /LPDDR4_DQS1P_A
- U1 pad N2: unconnected-(U1E-DDR_DQS1N_A/DDR4_DQSU_N_A/LPDDR4_DQS1N_A/DDR3_DQS1N/LPDDR3_DQS3N-PadN2) -> /LPDDR4_DQS1N_A
- U1 pad P2: unconnected-(U1E-DDR_DQ8_A/DDR4_DQU3_A/LPDDR4_DQ8_A/DDR3_DQ8/LPDDR3_DQ25-PadP2) -> /LPDDR4_DQ8_A
- U1 pad P37: unconnected-(U1G-AVSS1_3-PadP37) -> GNDREF
- U1 pad R1: unconnected-(U1E-DDR_DQ9_A/DDR4_DQU1_A/LPDDR4_DQ9_A/DDR3_DQ9/LPDDR3_DQ24-PadR1) -> /LPDDR4_DQ9_A
- U1 pad R2: unconnected-(U1E-DDR_DQ10_A/DDR4_DQU7_A/LPDDR4_DQ10_A/DDR3_DQ10/LPDDR3_DQ28-PadR2) -> /LPDDR4_DQ10_A
- U1 pad T2: unconnected-(U1E-DDR_DQ11_A/DDR4_DQU5_A/LPDDR4_DQ11_A/DDR3_DQ11/LPDDR3_DQ29-PadT2) -> /LPDDR4_DQ11_A
- U1 pad U2: unconnected-(U1H-VSS_16-PadU2) -> GNDREF
- U1 pad U37: unconnected-(U1G-AVSS1_4-PadU37) -> GNDREF
- U1 pad W2: unconnected-(U1H-VSS_17-PadW2) -> GNDREF
- U1 pad Y37: unconnected-(U1G-AVSS1_5-PadY37) -> GNDREF
