File: memory.kicad_sch (KiCad schematic)
At the start: 1 part, among them U1 RK3566

Commit message: initial commit
Parts:
- removed U1: RK3566, companion-computer:IC_RK3566, symbol RK3566:RK3566
- added C10, C11, C12, C13, C8, C9: 100 nF, symbol Device:C
- added C14, C15, C16, C17: 4.7 μF, symbol Device:C
- added R14: 240R, symbol Device:R
- added U1: RK3566, companion-computer:IC_RK3566, symbol RK3566:RK3566
Connections:
- new net: R14.1, U1.1F3 (DDR_RZQ)
- new net GNDREF: C10.2, C11.2, C12.2, C13.2, C14.2, C15.2, C16.2, C17.2, C8.2, C9.2, R14.2, U1.1D4 (DDR_AVSS)
- new net LPDDR4_A0_A: U1.C2 (DDR4_A11/LPDDR4_A0_A/DDR3_A7/LPDDR3_A8/AC11)
- new net LPDDR4_A0_B: U1.A9 (DDR4_A13/LPDDR4_A0_B/DDR3_A14/LPDDR3_A0/AC13)
- new net LPDDR4_A1_A: U1.C1 (DDR4_A2/LPDDR4_A1_A/DDR3_A4/LPDDR3_A6/AC2)
- new net LPDDR4_A1_B: U1.B9 (DDR4_A6/LPDDR4_A1_B/DDR3_A13/LPDDR3_A1/AC6)
- new net LPDDR4_A2_A: U1.1C1 (DDR4_A15_~{CAS}/LPDDR4_A2_A/DDR3_A0/-/AC15)
- new net LPDDR4_A2_B: U1.1B7 (DDR4_BA0/LPDDR4_A2_B/DDR3_A1/-/AC18)
- new net LPDDR4_A3_A: U1.1B3 (DDR4_A12/LPDDR4_A3_A/DDR3_BA2/-/AC12)
- new net LPDDR4_A3_B: U1.1B6 (DDR4_A4/LPDDR4_A3_B/DDR3_BA1/LPDDR3_A3/AC4)
- new net LPDDR4_A4_A: U1.1B1 (DDR4_A14_~{WE}/LPDDR4_A4_A/DDR3_A15/LPDDR3_A5/AC14)
- new net LPDDR4_A4_B: U1.1A6 (DDR4_BA1/LPDDR4_A4_B/DDR3_A12/LPDDR3_A4/AC19)
- new net LPDDR4_A5_A: U1.1A1 (DDR4_A16_~{RAS}/LPDDR4_A5_A/DDR3_~{RAS}/LPDDR3_A7/AC16)
- new net LPDDR4_A5_B: U1.B8 (DDR4_A5/LPDDR4_A5_B/DDR3_A11/LPDDR3_A2/AC5)
- new net LPDDR4_CKE0_A: U1.B4 (DDR4_CKE/LPDDR4_CKE0_A/DDR3_CKE/LPDDR3_CKE/AC22)
- new net LPDDR4_CKE0_B: U1.1A3 (DDR4_A10/LPDDR4_CKE0_B/DDR3_A10/-/AC10)
- new net LPDDR4_CKE1_A: U1.1C3 (DDR4_A3/LPDDR4_CKE1_A/DDR3_A3/-/AC3)
- new net LPDDR4_CKE1_B: U1.1A2 (DDR4_~{ACT}/LPDDR4_CKE1_B/DDR3_~{CAS}/-/AC17)
- new net LPDDR4_CLKN_A: U1.B5 (DDR4_CLKN/LPDDR4_CLKN_A/DDR3_CLKN/LPDDR3_CLKN/AC24)
- new net LPDDR4_CLKN_B: U1.B7 (DDR4_A9/LPDDR4_CLKN_B/DDR3_A5/-/AC9)
- new net LPDDR4_CLKP_A: U1.A5 (DDR4_CLKP/LPDDR4_CLKP_A/DDR3_CLKP/LPDDR3_CLKP/AC23)
- new net LPDDR4_CLKP_B: U1.A7 (DDR4_A0/LPDDR4_CLKP_B/DDR3_A9/-/AC0)
- new net LPDDR4_CS0_A: U1.B3 (DDR4_~{CS0}/LPDDR4_~{CS0}_A/DDR3_ODT1/LPDDR3_ODT0/AC25)
- new net LPDDR4_CS0_B: U1.1B5 (DDR4_ODT1/LPDDR4_~{CS0}_B/DDR3_~{CS0}/LPDDR3_~{CS0}/AC28)
- new net LPDDR4_CS1_A: U1.A3 (DDR4_~{CS1}/LPDDR4_~{CS1}_A/DDR3_~{CS1}/LPDDR3_ODT1/AC26)
- new net LPDDR4_CS1_B: U1.1A5 (DDR4_ODT0/LPDDR4_~{CS1}_B/DDR3_ODT0/LPDDR3_~{CS1}/AC27)
- new net LPDDR4_DM0_A: U1.1E2 (DDR_DM0_A/DDR4_DML_A/LPDDR4_DM0_A/DDR3_DM0/LPDDR3_DM1)
- new net LPDDR4_DM0_B: U1.1B8 (DDR_DM0_B/DDR4_DMU_B/LPDDR4_DM0_B/DDR3_DM2/LPDDR3_DM0)
- new net LPDDR4_DM1_A: U1.1G1 (DDR_DM1_A/DDR4_DMU_A/LPDDR4_DM1_A/DDR3_DM1/LPDDR3_DM3)
- new net LPDDR4_DM1_B: U1.1A11 (DDR_DM1_B/DDR4_DML_B/LPDDR4_DM1_B/DDR3_DM3/LPDDR3_DM2)
- new net LPDDR4_DQ0_A: U1.G2 (DDR_DQ0_A/DDR4_DQL0_A/LPDDR4_DQ0_A/DDR3_DQ0/LPDDR3_DQ15)
- new net LPDDR4_DQ0_B: U1.B12 (DDR_DQ0_B/DDR4_DQU7_B/LPDDR4_DQ0_B/DDR3_DQ16/LPDDR3_DQ1)
- new net LPDDR4_DQ10_A: U1.R2 (DDR_DQ10_A/DDR4_DQU7_A/LPDDR4_DQ10_A/DDR3_DQ10/LPDDR3_DQ28)
- new net LPDDR4_DQ10_B: U1.A20 (DDR_DQ10_B/DDR4_DQL4_B/LPDDR4_DQ10_B/DDR3_DQ26/LPDDR3_DQ22)
- new net LPDDR4_DQ11_A: U1.T2 (DDR_DQ11_A/DDR4_DQU5_A/LPDDR4_DQ11_A/DDR3_DQ11/LPDDR3_DQ29)
- new net LPDDR4_DQ11_B: U1.B20 (DDR_DQ11_B/DDR4_DQL6_B/LPDDR4_DQ11_B/DDR3_DQ27/LPDDR3_DQ23)
- new net LPDDR4_DQ12_A: U1.M1 (DDR_DQ12_A/DDR4_DQU2_A/LPDDR4_DQ12_A/DDR3_DQ12/LPDDR3_DQ26)
- new net LPDDR4_DQ12_B: U1.A15 (DDR_DQ12_B/DDR4_DQL7_B/LPDDR4_DQ12_B/DDR3_DQ28/LPDDR3_DQ16)
- new net LPDDR4_DQ13_A: U1.1F2 (DDR_DQ13_A/DDR4_DQU4_A/LPDDR4_DQ13_A/DDR3_DQ13/LPDDR3_DQ31)
- new net LPDDR4_DQ13_B: U1.B15 (DDR_DQ13_B/DDR4_DQL5_B/LPDDR4_DQ13_B/DDR3_DQ29/LPDDR3_DQ17)
- new net LPDDR4_DQ14_A: U1.1F1 (DDR_DQ14_A/DDR4_DQU6_A/LPDDR4_DQ14_A/DDR3_DQ14/LPDDR3_DQ30)
- new net LPDDR4_DQ14_B: U1.1C10 (DDR_DQ14_B/DDR4_DQL1_B/LPDDR4_DQ14_B/DDR3_DQ30/LPDDR3_DQ20)
- new net LPDDR4_DQ15_A: U1.1G2 (DDR_DQ15_A/DDR4_DQU0_A/LPDDR4_DQ15_A/DDR3_DQ15/LPDDR3_DQ27)
- new net LPDDR4_DQ15_B: U1.B16 (DDR_DQ15_B/DDR4_DQL3_B/LPDDR4_DQ15_B/DDR3_DQ31/LPDDR3_DQ21)
- new net LPDDR4_DQ1_A: U1.F2 (DDR_DQ1_A/DDR4_DQL2_A/LPDDR4_DQ1_A/DDR3_DQ1/LPDDR3_DQ14)
- new net LPDDR4_DQ1_B: U1.B10 (DDR_DQ1_B/DDR4_DQU5_B/LPDDR4_DQ1_B/DDR3_DQ17/LPDDR3_DQ5)
- new net LPDDR4_DQ2_A: U1.F1 (DDR_DQ2_A/DDR4_DQL4_A/LPDDR4_DQ2_A/DDR3_DQ2/LPDDR3_DQ10)
- new net LPDDR4_DQ2_B: U1.1A8 (DDR_DQ2_B/DDR4_DQU3_B/LPDDR4_DQ2_B/DDR3_DQ18/LPDDR3_DQ6)
- new net LPDDR4_DQ3_A: U1.E1 (DDR_DQ3_A/DDR4_DQL6_A/LPDDR4_DQ3_A/DDR3_DQ3/LPDDR3_DQ9)
- new net LPDDR4_DQ3_B: U1.1A7 (DDR_DQ3_B/DDR4_DQU1_B/LPDDR4_DQ3_B/DDR3_DQ19/LPDDR3_DQ4)
- new net LPDDR4_DQ4_A: U1.M2 (DDR_DQ4_A/DDR4_DQL7_A/LPDDR4_DQ4_A/DDR3_DQ4/LPDDR3_DQ13)
- new net LPDDR4_DQ4_B: U1.B13 (DDR_DQ4_B/DDR4_DQU0_B/LPDDR4_DQ4_B/DDR3_DQ20/LPDDR3_DQ2)
- new net LPDDR4_DQ5_A: U1.K1 (DDR_DQ5_A/DDR4_DQL5_A/LPDDR4_DQ5_A/DDR3_DQ5/LPDDR3_DQ12)
- new net LPDDR4_DQ5_B: U1.1A10 (DDR_DQ5_B/DDR4_DQU6_B/LPDDR4_DQ5_B/DDR3_DQ21/LPDDR3_DQ3)
- new net LPDDR4_DQ6_A: U1.K2 (DDR_DQ6_A/DDR4_DQL3_A/LPDDR4_DQ6_A/DDR3_DQ6/LPDDR3_DQ8)
- new net LPDDR4_DQ6_B: U1.1B9 (DDR_DQ6_B/DDR4_DQU4_B/LPDDR4_DQ6_B/DDR3_DQ22/LPDDR3_DQ7)
- new net LPDDR4_DQ7_A: U1.1E1 (DDR_DQ7_A/DDR4_DQL1_A/LPDDR4_DQ7_A/DDR3_DQ7/LPDDR3_DQ11)
- new net LPDDR4_DQ7_B: U1.1A9 (DDR_DQ7_B/DDR4_DQU2_B/LPDDR4_DQ7_B/DDR3_DQ23/LPDDR3_DQ0)
- new net LPDDR4_DQ8_A: U1.P2 (DDR_DQ8_A/DDR4_DQU3_A/LPDDR4_DQ8_A/DDR3_DQ8/LPDDR3_DQ25)
- new net LPDDR4_DQ8_B: U1.B19 (DDR_DQ8_B/DDR4_DQL0_B/LPDDR4_DQ8_B/DDR3_DQ24/LPDDR3_DQ18)
- new net LPDDR4_DQ9_A: U1.R1 (DDR_DQ9_A/DDR4_DQU1_A/LPDDR4_DQ9_A/DDR3_DQ9/LPDDR3_DQ24)
- new net LPDDR4_DQ9_B: U1.A19 (DDR_DQ9_B/DDR4_DQL2_B/LPDDR4_DQ9_B/DDR3_DQ25/LPDDR3_DQ19)
- new net LPDDR4_DQS0N_A: U1.H1 (DDR_DQS0N_A/DDR4_DQSL_N_A/LPDDR4_DQS0N_A/DDR3_DQS0N/LPDDR3_DQS1N)
- new net LPDDR4_DQS0N_B: U1.A12 (DDR_DQS0N_B/DDR4_DQSU_N_B/LPDDR4_DQS0N_B/DDR3_DQS2N/LPDDR3_DQS0N)
- new net LPDDR4_DQS0P_A: U1.H2 (DDR_DQS0P_A/DDR4_DQSL_P_A/LPDDR4_DQS0P_A/DDR3_DQS0P/LPDDR3_DQS1P)
- new net LPDDR4_DQS0P_B: U1.A13 (DDR_DQS0P_B/DDR4_DQSU_P_B/LPDDR4_DQS0P_B/DDR3_DQS2P/LPDDR3_DQS0P)
- new net LPDDR4_DQS1N_A: U1.N2 (DDR_DQS1N_A/DDR4_DQSU_N_A/LPDDR4_DQS1N_A/DDR3_DQS1N/LPDDR3_DQS3N)
- new net LPDDR4_DQS1N_B: U1.B17 (DDR_DQS1N_B/DDR4_DQSL_N_B/LPDDR4_DQS1N_B/DDR3_DQS3N/LPDDR3_DQS2N)
- new net LPDDR4_DQS1P_A: U1.N1 (DDR_DQS1P_A/DDR4_DQSU_P_A/LPDDR4_DQS1P_A/DDR3_DQS1P/LPDDR3_DQS3P)
- new net LPDDR4_DQS1P_B: U1.A17 (DDR_DQS1P_B/DDR4_DQSL_P_B/LPDDR4_DQS1P_B/DDR3_DQS3P/LPDDR3_DQS2P)
- new net LPDDR4_ODT0_CA_A: U1.E2 (DDR4_A8/LPDDR4_ODT0_CA_A/DDR3_A6/LPDDR3_A9/AC8)
- new net LPDDR4_ODT0_CA_B: U1.A10 (DDR4_A7/LPDDR4_ODT0_CA_B/DDR3_A8/-/AC7)
- new net LPDDR4_RESET: U1.1C7 (DDR4_~{RESET}/LPDDR4_~{RESET}/DDR3_~{RESET}/AC29)
- new net VCC0V6_DDR: C11.1, C13.1, C15.1, C17.1, C9.1, U1.1E6 (DDRPHY_VDDQL_1), U1.1E7 (DDRPHY_VDDQL_2), U1.1E9 (DDRPHY_VDDQL_3), U1.1F5 (DDRPHY_VDDQL_4), U1.1G5 (DDRPHY_VDDQL_5)
- new net VCC_DDR: C10.1, C12.1, C14.1, C16.1, C8.1, U1.1D5 (DDRPHY_VDDQ_1), U1.1D6 (DDRPHY_VDDQ_2), U1.1D7 (DDRPHY_VDDQ_3), U1.1D8 (DDRPHY_VDDQ_4), U1.1D9 (DDRPHY_VDDQ_5), U1.1E4 (DDRPHY_VDDQ_6), U1.1F4 (DDRPHY_VDDQ_7), U1.1G4 (DDRPHY_VDDQ_8)
- no-connect marks 0 -> 4
Other:
- removed sheet Memory
- removed sheet Power Management IC
- removed sheet Power and Ground
