File: power_management.kicad_sch (KiCad schematic)
At the start: 43 parts, among them U3 RK3566, U4 MP9943GQ-Z, U5 MP9943GQ-Z

Commit message: pmic
Parts:
- added C18, C19: 100nF, symbol Device:C
- added Q1: NMOS, symbol Simulation_SPICE:NMOS
- added U6: NCV68061SNAIT1G, companion-computer:TSOP-6_L3.0-W1.5-P0.95-BL, symbol RK3566:NCV68061SNAIT1G
Connections:
- net GNDREF: now also C18.2, C19.2, U6.2 (GND)
- net +5V renamed +3.8V
- net +3.8V: no longer C57.1, C58.1, L1.2, R9.2
- new net: Q1.2 (G), U6.5 (G)
- new net +5V BAT: C18.1, C57.1, C58.1, L1.2, Q1.1 (D), R9.2, U6.6 (S)
- new net +5V SYS: C19.1, Q1.3 (S), U6.4 (D)
Other:
- note added: "POWER IDEAL DIODE"
